File: PCB_Buzzer_withNPN_MountingHoles_newRFID_1layer/PXB_buzzer_noAmpli.kicad_pcb (KiCad board)
At the start: 2 copper layers, 86.4 x 99.1 mm, 15 parts, among them J1 Conn_01x08, Q1 EBC, U1 NodeMCU_1.0, Y1 YWRobot

Commit message: ywrobot moved
Parts:
- moved Y1 9.00 mm to (143.0, 47.9)
Routing:
- net Net-(R3-Pad2): track 63.0 -> 72.2 mm
- net /GND->5(GND): track 326.3 -> 328.1 mm
